Commit message: Imported upstream version '0.0.6' of 'upstream'

File: evarobot_description/urdf/evarobot.urdf.xacro (robot description, xacro)
@@ -6,4 +6,5 @@
   <xacro:property name="pi" value="3.1415926535897931" />
   <!-- Includes -->
+  <xacro:include filename="$(find evarobot_description)/urdf/materials.urdf.xacro"/>
   <xacro:include filename="$(find evarobot_description)/urdf/evarobot_base.urdf.xacro"/>
   <xacro:include filename="$(find evarobot_description)/urdf/evarobot_caster.urdf.xacro"/>
@@ -25,5 +26,4 @@
 		<publishWheelJointState>true</publishWheelJointState>
 		<wheelAcceleration>1</wheelAcceleration>
-	  <!--  Plugin arkadan suruslu robotlar icin yapildigindan jointler ters yazildi  -->
 	  <leftJoint>right_wheel_joint</leftJoint>
 	  <rightJoint>left_wheel_joint</rightJoint>
@@ -33,5 +33,5 @@
 	  <commandTopic>cmd_vel</commandTopic>
 	  <odometryTopic>odom</odometryTopic>
-	  <odometryFrame>odom</odometryFrame>
+	  <odometryFrame>odom_combined</odometryFrame>
     </plugin>
   </gazebo>
@@ -43,5 +43,5 @@
 					   mesh_x="0.065"
 					   mesh_y="-0.11"
-					   mesh_z="-0.20"
+					   mesh_z="-0.15"
 					   mesh_roll="0.0"
 					   mesh_pitch="0.0"
@@ -54,5 +54,5 @@
 						joint_x="0.0"
 						joint_y="0.16"
-						joint_z="-0.1685"
+						joint_z="${-0.15 + (85-54)/1000}"
 						joint_roll="0.0"
 						joint_pitch="0.0"
@@ -65,5 +65,5 @@
 						joint_x="0.0"
 						joint_y="-0.16"
-						joint_z="-0.1685"
+						joint_z="${-0.15 + (85-54)/1000}"
 						joint_roll="0.0"
 						joint_pitch="0.0"
@@ -77,6 +77,6 @@
 						 x="0.1604"
 						 y="0.0"
-						 z="-0.228"
-						 roll="-1.57075"
+						 z="${-0.15 -13.5/2000}"
+						 roll="0.0"
 						 pitch="0.0"
 						 yaw="0.0"
@@ -89,6 +89,6 @@
 						 x="-0.1604"
 						 y="0.0"
-						 z="-0.228"
-						 roll="-1.57075"
+						 z="${-0.15 -13.5/2000}"
+						 roll="0.0"
 						 pitch="0.0"
 						 yaw="0.0"
@@ -98,8 +98,8 @@
 						 parent_link="base_link" />
   <!-- Lidar -->
-  <xacro:evarobot_lidar prefix="sensor/lidar"
+  <xacro:evarobot_lidar prefix="lidar"
                         joint_x="-0.15"
                         joint_y="0.0"
-                        joint_z="0.4415"
+                        joint_z="${0.4415 + 100/1000}"
                         joint_roll="0.0"
                         joint_pitch="0.0"
@@ -117,18 +117,187 @@
 												topic_name="lidar"
 												frame_name="lidar_link" />
-<!-- joint_yaw="-1.5708" -->
   <!-- Kinect -->
-   <xacro:evarobot_kinect prefix="sensor/kinect"
+   <xacro:evarobot_kinect prefix="kinect"
 						 joint_x="0.17"
 						 joint_y="0.0"
-						 joint_z="0.16"
-						 joint_roll="0"
+						 joint_z="${0.21 - 18.7/1000}"
+						 joint_roll="0.0"
 						 joint_pitch="0.0"
-						 joint_yaw="0"
+						 joint_yaw="0.0"
 						 parent_link="base_link"
 						 base_line="0.2"
 						 update_rate="1.0"
 						 camera_name="camera" />
-  <!-- Bumper -->
+  <!-- AHRS/IMU -->
+  <xacro:evarobot_ahrs prefix="imu"
+					   joint_x="0.0"
+					   joint_y="0.0"
+					   joint_z="0.19"
+					   joint_roll="${pi}"
+					   joint_pitch="0.0"
+					   joint_yaw="0.0"
+					   parent_link="base_link"
+					   topic_name="imu"
+					   frame_name="imu_link"
+					   update_rate="10.0"
+					   service_name="imu_service"
+					   robot_namespace="evarobot" />
+ <!-- Sonar -->
+	<xacro:evarobot_sonar prefix="sonar0"
+				parent_link="base_link"
+				scan_samples="320"
+				scan_resolution="1"
+				min_angle="-0.479965544"
+				max_angle="0.479965544"
+				range_resolution="0.01"
+				min_range="0.02"
+				max_range="5.0"
+				topic_name="sonar0"
+				frame_name="sonar0_link"
+				update_rate="4" >
+				<origin xyz="0.130 -0.147 ${0.03+50/1000}" rpy="0 0 ${-pi/3}" />
+	</xacro:evarobot_sonar>
+  <xacro:evarobot_sonar prefix="sonar1"
+						parent_link="base_link"
+						scan_samples="320"
+						scan_resolution="1"
+						min_angle="-0.479965544"
+						max_angle="0.479965544"
+						range_resolution="0.01"
+						min_range="0.02"
+						max_range="5.0"
+						topic_name="sonar1"
+						frame_name="sonar1_link"
+						update_rate="4">
+								<origin xyz="0.213 0.0 ${0.03+50/1000}" rpy="0 0 0" />
+	</xacro:evarobot_sonar>
+	<xacro:evarobot_sonar prefix="sonar2"
+				parent_link="base_link"
+				scan_samples="320"
+				scan_resolution="1"
+				min_angle="-0.479965544"
+				max_angle="0.479965544"
+				range_resolution="0.01"
+				min_range="0.02"
+				max_range="5.0"
+				topic_name="sonar2"
+				frame_name="sonar2_link"
+				update_rate="4" >
+				<origin xyz="0.130 0.147 ${0.03+50/1000}" rpy="0 0 ${pi/3}" />
+	</xacro:evarobot_sonar>
+	<xacro:evarobot_sonar prefix="sonar3"
+					parent_link="base_link"
+					scan_samples="320"
+					scan_resolution="1"
+					min_angle="-0.479965544"
+					max_angle="0.479965544"
+					range_resolution="0.01"
+					min_range="0.02"
+					max_range="5.0"
+					topic_name="sonar3"
+					frame_name="sonar3_link"
+					update_rate="4">
+						<origin xyz="-0.045 0.168 ${0.03+50/1000}" rpy="0 0 ${pi/2}" />
+	</xacro:evarobot_sonar>
+	<xacro:evarobot_sonar prefix="sonar4"
+					parent_link="base_link"
+					scan_samples="320"
+					scan_resolution="1"
+					min_angle="-0.479965544"
+					max_angle="0.479965544"
+					range_resolution="0.01"
+					min_range="0.02"
+					max_range="5.0"
+					topic_name="sonar4"
+					frame_name="sonar4_link"
+					update_rate="4" >
+					<origin xyz="-0.191 0.084 ${0.03+50/1000}" rpy="0 0 ${5*pi/6}" />
+	</xacro:evarobot_sonar>
+	<xacro:evarobot_sonar prefix="sonar5"
+					parent_link="base_link"
+					scan_samples="320"
+					scan_resolution="1"
+					min_angle="-0.479965544"
+					max_angle="0.479965544"
+					range_resolution="0.01"
+					min_range="0.02"
+					max_range="5.0"
+					topic_name="sonar5"
+					frame_name="sonar5_link"
+					update_rate="4" >
+					<origin xyz="-0.191 -0.084 ${0.03+50/1000}" rpy="0 0 ${-5*pi/6}" />
+	</xacro:evarobot_sonar>
+  <xacro:evarobot_sonar prefix="sonar6"
+						parent_link="base_link"
+						scan_samples="320"
+						scan_resolution="1"
+						min_angle="-0.479965544"
+						max_angle="0.479965544"
+						range_resolution="0.01"
+						min_range="0.02"
+						max_range="5.0"
+						topic_name="sonar6"
+						frame_name="sonar6_link"
+						update_rate="4">
+						  <origin xyz="-0.045 -0.168 ${0.03+50/1000}" rpy="0 0 ${-pi/2}" />
+  </xacro:evarobot_sonar>
+  <!-- Infrared -->
+  <xacro:evarobot_infrared prefix="ir0"
+						   parent_link="base_link"
+						   scan_samples="320"
+						   scan_resolution="1"
+						   min_angle="-0.001"
+						   max_angle="0.001"
+						   range_resolution="0.01"
+						   min_range="0.10"
+						   max_range="0.80"
+						   topic_name="ir0"
+						   frame_name="ir0_link"
+						   update_rate="4" >
+						   	     <origin xyz="0.191 -0.084 ${-0.122+50/1000}" rpy="0 0 ${-pi/6}" />
+	</xacro:evarobot_infrared>
+  <xacro:evarobot_infrared prefix="ir1"
+						   parent_link="base_link"
+						   scan_samples="320"
+						   scan_resolution="1"
+						   min_angle="-0.001"
+						   max_angle="0.001"
+						   range_resolution="0.01"
+						   min_range="0.10"
+						   max_range="0.80"
+						   topic_name="ir1"
+						   frame_name="ir1_link"
+						   update_rate="4">
+						   		<origin xyz="0.191 0.084 ${-0.122+50/1000}" rpy="0 0 ${pi/6}" />
+	</xacro:evarobot_infrared>
+  <xacro:evarobot_infrared prefix="ir2"
+						   parent_link="base_link"
+						   scan_samples="320"
+						   scan_resolution="1"
+						   min_angle="-0.001"
+						   max_angle="0.001"
+						   range_resolution="0.01"
+						   min_range="0.10"
+						   max_range="0.80"
+						   topic_name="ir2"
+						   frame_name="ir2_link"
+						   update_rate="4">
+						   		<origin xyz="-0.130 0.147 ${-0.122+50/1000}" rpy="0 0 ${2*pi/3}" />
+	</xacro:evarobot_infrared>
+  <xacro:evarobot_infrared prefix="ir3"
+						   parent_link="base_link"
+						   scan_samples="320"
+						   scan_resolution="1"
+						   min_angle="-0.001"
+						   max_angle="0.001"
+						   range_resolution="0.01"
+						   min_range="0.10"
+						   max_range="0.80"
+						   topic_name="ir3"
+						   frame_name="ir3_link"
+						   update_rate="4">
+						   	    <origin xyz="-0.130 -0.147 ${-0.122+50/1000}" rpy="0 0 ${-2*pi/3}" />
+	</xacro:evarobot_infrared>
+ <!-- Bumper -->
   <xacro:evarobot_bumper prefix="bumper0"
 						 box_x="0.015"
@@ -139,5 +308,5 @@
 						 topic_name="bumper0"
 						 frame_name="bumper0_link" >
-  <origin xyz="0.191 -0.084 -0.122" rpy="0 0 ${-pi/6}" />
+  <origin xyz="0.191 -0.084 ${-0.122+50/1000}" rpy="0 0 ${-pi/6}" />
 						 </xacro:evarobot_bumper>
   <xacro:evarobot_bumper prefix="bumper1"
@@ -149,6 +318,5 @@
 						 topic_name="bumper1"
 						 frame_name="bumper1_link" >
-						   <origin xyz="0.213 0.0 -0.122" rpy="0 0 0" />
-  <origin xyz="0.213 0.0 -0.122" rpy="0 0 0" />
+						   <origin xyz="0.213 0.0 ${-0.122+50/1000}" rpy="0 0 0" />
 						</xacro:evarobot_bumper>
   <xacro:evarobot_bumper prefix="bumper2"
@@ -160,176 +328,5 @@
 						 topic_name="bumper2"
 						 frame_name="bumper2_link" >
-  <origin xyz="0.191 0.084 -0.122" rpy="0 0 ${pi/6}" />
+  <origin xyz="0.191 0.084 ${-0.122+50/1000}" rpy="0 0 ${pi/6}" />
 						 </xacro:evarobot_bumper>
-  <!-- AHRS/IMU
-  <xacro:evarobot_ahrs prefix="sensor/imu"
-					   joint_x="0.0"
-					   joint_y="0.0"
-					   joint_z="0.19"
-					   joint_roll="0.0"
-					   joint_pitch="0.0"
-					   joint_yaw="0.0"
-					   parent_link="base_link"
-					   topic_name="imu"
-					   frame_name="sensor/imu_link"
-					   update_rate="10.0"
-					   service_name="imu_service"
-					   robot_namespace="evarobot" />
-	-->
- <!-- Sonar -->
-	<xacro:evarobot_sonar prefix="sensor/sonar0"
-				parent_link="base_link"
-				scan_samples="320"
-				scan_resolution="1"
-				min_angle="-0.479965544"
-				max_angle="0.479965544"
-				range_resolution="0.01"
-				min_range="0.02"
-				max_range="5.0"
-				topic_name="sonar0"
-				frame_name="sensor/sonar0_link"
-				update_rate="4" >
-				<origin xyz="0.130 -0.147 0.03" rpy="0 0 ${-pi/3}" />
-	</xacro:evarobot_sonar>
-  <xacro:evarobot_sonar prefix="sensor/sonar1"
-						parent_link="base_link"
-						scan_samples="320"
-						scan_resolution="1"
-						min_angle="-0.479965544"
-						max_angle="0.479965544"
-						range_resolution="0.01"
-						min_range="0.02"
-						max_range="5.0"
-						topic_name="sonar1"
-						frame_name="sensor/sonar1_link"
-						update_rate="4">
-								<origin xyz="0.213 0.0 0.03" rpy="0 0 0" />
-	</xacro:evarobot_sonar>
-	<xacro:evarobot_sonar prefix="sensor/sonar2"
-				parent_link="base_link"
-				scan_samples="320"
-				scan_resolution="1"
-				min_angle="-0.479965544"
-				max_angle="0.479965544"
-				range_resolution="0.01"
-				min_range="0.02"
-				max_range="5.0"
-				topic_name="sonar2"
-				frame_name="sensor/sonar2_link"
-				update_rate="4" >
-				<origin xyz="0.130 0.147 0.03" rpy="0 0 ${pi/3}" />
-	</xacro:evarobot_sonar>
-	<xacro:evarobot_sonar prefix="sensor/sonar3"
-					parent_link="base_link"
-					scan_samples="320"
-					scan_resolution="1"
-					min_angle="-0.479965544"
-					max_angle="0.479965544"
-					range_resolution="0.01"
-					min_range="0.02"
-					max_range="5.0"
-					topic_name="sonar3"
-					frame_name="sensor/sonar3_link"
-					update_rate="4">
-						<origin xyz="-0.045 0.168 0.03" rpy="0 0 ${pi/2}" />
-	</xacro:evarobot_sonar>
-	<xacro:evarobot_sonar prefix="sensor/sonar4"
-					parent_link="base_link"
-					scan_samples="320"
-					scan_resolution="1"
-					min_angle="-0.479965544"
-					max_angle="0.479965544"
-					range_resolution="0.01"
-					min_range="0.02"
-					max_range="5.0"
-					topic_name="sonar4"
-					frame_name="sensor/sonar4_link"
-					update_rate="4" >
-					<origin xyz="-0.191 0.084 0.03" rpy="0 0 ${5*pi/6}" />
-	</xacro:evarobot_sonar>
-	<xacro:evarobot_sonar prefix="sensor/sonar5"
-					parent_link="base_link"
-					scan_samples="320"
-					scan_resolution="1"
-					min_angle="-0.479965544"
-					max_angle="0.479965544"
-					range_resolution="0.01"
-					min_range="0.02"
-					max_range="5.0"
-					topic_name="sonar5"
-					frame_name="sensor/sonar5_link"
-					update_rate="4" >
-					<origin xyz="-0.191 -0.084 0.03" rpy="0 0 ${-5*pi/6}" />
-	</xacro:evarobot_sonar>
-  <xacro:evarobot_sonar prefix="sensor/sonar6"
-						parent_link="base_link"
-						scan_samples="320"
-						scan_resolution="1"
-						min_angle="-0.479965544"
-						max_angle="0.479965544"
-						range_resolution="0.01"
-						min_range="0.02"
-						max_range="5.0"
-						topic_name="sonar6"
-						frame_name="sensor/sonar6_link"
-						update_rate="4">
-						  <origin xyz="-0.045 -0.168 0.03" rpy="0 0 ${-pi/2}" />
-  </xacro:evarobot_sonar>
-  <!-- Infrared -->
-  <xacro:evarobot_infrared prefix="sensor/ir0"
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
File: evarobot_description/urdf/evarobot_ahrs.urdf.xacro (robot description, xacro)
@@ -6,5 +6,5 @@
 				<mass value="0.001"/>
 				<origin rpy="0 0 0" xyz="0 0 0"/>
-				<inertia ixx="0.0001" ixy="0" ixz="0" iyy="0.000001" iyz="0" izz="0.0001"/>
+				<inertia ixx="0.0001" ixy="0" ixz="0" iyy="0.0001" iyz="0" izz="0.0001"/>
 			</inertial>
 			<visual>
@@ -30,5 +30,5 @@
 			<plugin name="${prefix}_plugin" filename="libgazebo_ros_imu.so">
 				<alwaysOn>true</alwaysOn>
-				<robotNamespace>gazebo</robotNamespace>
+		<!--		<robotNamespace>gazebo</robotNamespace>     -->
 				<frameName>${frame_name}</frameName>
 				<bodyName>${prefix}_link</bodyName>

File: evarobot_description/urdf/evarobot_base.urdf.xacro (robot description, xacro)
@@ -5,8 +5,6 @@
 			<collision>
 				<origin xyz="0 0 0" rpy="0 0 0"/>
-				<!--<origin xyz="${mesh_x} ${mesh_y} ${mesh_z}" rpy="${mesh_roll} ${mesh_pitch} ${mesh_yaw}" /> -->
 				<geometry>
-<!--					<mesh filename="package://evarobot_description/meshes/eva50.stl" scale="0.01 0.01 0.01"/>   -->
-				<box size="${box_x} ${box_y} ${box_z}"/>
+					<box size="${box_x} ${box_y} ${box_z}"/>
 				</geometry>
 			</collision>
@@ -14,20 +12,52 @@
 				<origin xyz="${mesh_x} ${mesh_y} ${mesh_z}" rpy="${mesh_roll} ${mesh_pitch} ${mesh_yaw}" />
 				<geometry>
-				<!-- <box size="${box_x} ${box_y} ${box_z}"/> -->
-					<mesh filename="package://evarobot_description/meshes/eva50.stl" scale="0.01 0.01 0.01"/>
+					<mesh filename="package://evarobot_description/meshes/base.stl" scale="1 1 1"/>
 				</geometry>
-				<material name="red">
-					<color rgba="0.4 0.7 .8 1"/>
-				</material>
+				<material name="Black" />
 			</visual>
 			<inertial>
 				<origin xyz="0 0 0" rpy="0 0 0"/>
-				<mass value="15"/>
+				<mass value="10.0"/>
 				<inertia
-					ixx="0.875" ixy="0.155" ixz="0.143"
-					iyy="0.155" iyz="0.143"
-					izz="0.143"/>
+					ixx="1.0" ixy="0" ixz="0"
+					iyy="1.0" iyz="0"
+					izz="1.0"/>
 			</inertial>
 		</link>
+		<gazebo reference="${prefix}_link">
+      <material>Gazebo/Black</material>
+		</gazebo>
+		<link name="${prefix}color_link">
+			<collision>
+				<origin xyz="0 0 0" rpy="0 0 0"/>
+				<geometry>
+					<box size="0.0001 0.0001 0.0001"/>
+				</geometry>
+			</collision>
+			<visual>
+				<origin xyz="${mesh_x} ${mesh_y} ${mesh_z}" rpy="${mesh_roll} ${mesh_pitch} ${mesh_yaw}" />
+				<geometry>
+					<mesh filename="package://evarobot_description/meshes/base_orange.stl" scale="1 1 1"/>
+				</geometry>
+				<material name="Orange" />
+			</visual>
+			<inertial>
+				<origin xyz="0 0 0" rpy="0 0 0"/>
+				<mass value="0.0001"/>
+				<inertia
+					ixx="1e-6" ixy="0.0" ixz="0.0"
+					iyy="1e-6" iyz="0.0"
+					izz="1e-6"/>
+			</inertial>
+		</link>
+		<gazebo reference="${prefix}color_link">
+      <material>Gazebo/Orange</material>
+		</gazebo>
+		<joint name="${prefix}color_joint" type="fixed">
+			<axis xyz="0 1 0" />
+			<origin xyz="0 0 0" rpy="0 0 0"/>
+			<parent link="${prefix}_link"/>
+			<child link="${prefix}color_link"/>
+		</joint>
 	</xacro:macro>
 </robot>

File: evarobot_description/urdf/evarobot_bumper.urdf.xacro (robot description, xacro)
@@ -18,10 +18,4 @@
 				</geometry>
 			</collision>
-			<visual>
-				<origin xyz="0 0 0" rpy="0 0 0"/>
-				<geometry>
-					<box size="${box_x} ${box_y} ${box_z}"/>
-				</geometry>
-			</visual>
 			<inertial>
 				<mass value="1e-5" />

File: evarobot_description/urdf/evarobot_caster.urdf.xacro (robot description, xacro)
@@ -2,36 +2,114 @@
 <robot xmlns:xacro="http://ros.org/wiki/xacro">
 	<xacro:macro name="evarobot_caster" params="prefix radius x y z roll pitch yaw axis_x axis_y axis_z parent_link">
-		<link name="${prefix}_link">
+    <link name="${prefix}_base_link">
 			<collision>
 				<origin rpy="0 0 0" xyz="0 0 0"/>
 				<geometry>
-					<sphere radius="${radius}"/>
+					<box size="${60/1000} ${60/1000} ${13.5/1000}"/>
 				</geometry>
 			</collision>
 			<visual>
+				<origin rpy="${pi} 0 0" xyz="${-5/1000} ${-21.5/2000} ${13.5/2000}"/>
 				<geometry>
-					<sphere radius="${radius}"/>
+					<mesh filename="package://evarobot_description/meshes/caster_base.stl" scale="1 1 1"/>
 				</geometry>
-				<material name="black">
-					<color rgba="0 0 0 1"/>
-				</material>
+				<material name="Grey"/>
 			</visual>
 			<inertial>
-				<origin xyz="0 0 0" rpy="0 0 0"/>
-				<mass value="0.5"/>
-				<inertia ixx="1e-1" ixy="0" ixz="0" iyy="1e-1" iyz="0" izz="1e-1" />
+				<mass value="0.01" />
+				<origin xyz="0 0 0" />
+				<inertia ixx="1e-6" ixy="0.0" ixz="0.0"
+								 iyy="1e-6" iyz="0.0"
+								 izz="1e-6" />
 			</inertial>
 		</link>
-		<gazebo reference="${prefix}_link">
-			<mu1>0.2</mu1>
-			<mu2>0.2</mu2>
+		<gazebo reference="${prefix}_base_link">
+			<material>Gazebo/Grey</material>
+	    <mu1>0.0</mu1>
+	    <mu2>0.0</mu2>
+	    <kp>1000000.0</kp>
+	    <kd>100.0</kd>
+	    <minDepth>0.001</minDepth>
+	    <maxVel>1.0</maxVel>
 		</gazebo>
-		<joint name="${prefix}_joint" type="continuous">
+		<joint name="${prefix}_base_joint" type="fixed">
 			<parent link="${parent_link}"/>
-			<child link="${prefix}_link"/>
+			<child link="${prefix}_base_link"/>
 			<origin rpy="${roll} ${pitch} ${yaw}" xyz="${x} ${y} ${z}"/>
-			<axis xyz="${axis_x} ${axis_y} ${axis_z}"/>
-			<limit effort="10" velocity="10"/>
-			<joint_properties damping="0.0" friction="0.3"/>
+			<axis xyz="0 0 0"/>
+		</joint>
+    <link name="${prefix}_rotate_link">
+			<collision>
+				<origin rpy="0 0 0" xyz="0 0 0"/>
+				<geometry>
+					<cylinder length="${23/1000}" radius="${21.5/1000}"/>
+				</geometry>
+			</collision>
+			<visual>
+				<origin rpy="${pi} 0 ${pi/2}" xyz="0 0 ${10/1000}"/>
+				<geometry>
+					<mesh filename="package://evarobot_description/meshes/caster_rot.stl" scale="1 1 1"/>
+				</geometry>
+				<material name="Grey"/>
+			</visual>
+			<inertial>
+				<mass value="0.01" />
+				<origin xyz="0 0 0" />
+				<inertia ixx="1e-6" ixy="0.0" ixz="0.0"
+								 iyy="1e-6" iyz="0.0"
+								 izz="1e-6" />
+			</inertial>
+		</link>
+		<gazebo reference="${prefix}_rotate_link">
+			<material>Gazebo/Grey</material>
+	    <mu1>0.0</mu1>
+	    <mu2>0.0</mu2>
+	    <kp>1000000.0</kp>
+	    <kd>100.0</kd>
+	    <minDepth>0.001</minDepth>
+	    <maxVel>1.0</maxVel>
+		</gazebo>
+		<joint name="${prefix}_base_rotate_joint" type="continuous">
+			<parent link="${prefix}_base_link"/>
+			<child link="${prefix}_rotate_link"/>
+			<origin rpy="0 0 0" xyz="0.0 0.0 ${-37/2000}"/>
+			<axis xyz="0 0 1"/>
+		</joint>
+    <link name="${prefix}_wheel_link">
+			<collision>
+				<origin rpy="${pi/2} 0 0" xyz="0 0 0"/>
+				<geometry>
+					<sphere radius="${35/2000}"/>
+				</geometry>
+			</collision>
+			<visual>
+				<origin rpy="${pi/2} 0 0" xyz="0 0 0"/>
+				<geometry>
+					<sphere radius="${35/2000}"/>
+				</geometry>
+				<material name="Yellow"/>
+			</visual>
+			<inertial>
+				<mass value="0.01" />
+				<origin xyz="0 0 0" />
+				<inertia ixx="1e-6" ixy="0.0" ixz="0.0"
+								 iyy="1e-6" iyz="0.0"
+								 izz="1e-6" />
+			</inertial>
+		</link>
+		<gazebo reference="${prefix}_wheel_link">
+			<material>Gazebo/Yellow</material>
+			<mu1>0.0</mu1>
+	    <mu2>0.0</mu2>
+	    <kp>1000000.0</kp>
+	    <kd>100.0</kd>
+	    <minDepth>0.001</minDepth>
+	    <maxVel>1.0</maxVel>
+		</gazebo>
+		<joint name="${prefix}_rotate_wheel_joint" type="continuous">
+			<parent link="${prefix}_rotate_link"/>
+			<child link="${prefix}_wheel_link"/>
+			<origin rpy="0 0 0" xyz="${-14.632/1000} 0.0 ${-23/2000}"/>
+			<axis xyz="0.577350269 0.577350269 0.577350269"/>
 		</joint>
 	</xacro:macro>

File: evarobot_description/urdf/evarobot_infrared.urdf.xacro (robot description, xacro)
@@ -21,5 +21,5 @@
 				<mass value="0.001" />
 				<origin xyz="0 0 0" rpy="0 0 0" />
-				<inertia ixx="0.000000017" ixy="0" ixz="0" iyy="0.000000017" iyz="0" izz="0.000000017" />
+				<inertia ixx="1e-6" ixy="0" ixz="0" iyy="1e-6" iyz="0" izz="1e-6" />
 			</inertial>
 <!--
