Commit message: Imported upstream version '0.0.6' of 'upstream'

File: evarobot_description/urdf/evarobot_kinect.urdf.xacro (robot description, xacro)
@@ -8,75 +8,113 @@
 			camera_name
 			">
-		<!-- Kinect Link -->
-		<link name="${prefix}_link">
-			<collision>
-				<origin xyz="0 0 0" rpy="0 0 0"/>
-				<geometry>
-					<box size="0.1 0.1 0.1"/>
-				</geometry>
-			</collision>
-			<visual>
-				<origin xyz="0 0 0" rpy="0 0 0"/>
-				<geometry>
-					<mesh filename="package://evarobot_description/meshes/kinect.dae"/>
-				</geometry>
-			</visual>
-			<inertial>
-				<mass value="1e-5" />
-				<origin xyz="0 0 0" rpy="0 0 0"/>
-				<inertia ixx="1e-6" ixy="0" ixz="0" iyy="1e-6" iyz="0" izz="1e-6" />
-			</inertial>
-		</link>
-		<!-- Kinect Joint -->
-		<joint name="${prefix}_joint" type="fixed">
-			<axis xyz="0 1 0" />
+    <joint name="camera_rgb_joint" type="fixed">
+			<origin xyz="0.0 -0.02 0.0" rpy="0.0 0.0 0.0"/>
+			<parent link="camera_link"/>
+      <child link="camera_rgb_frame" />
+    </joint>
+    <link name="camera_rgb_frame"/>
+    <joint name="camera_rgb_optical_joint" type="fixed">
+      <origin xyz="0 0 0" rpy="${-pi/2} 0 ${-pi/2}" />
+      <parent link="camera_rgb_frame" />
+      <child link="camera_rgb_optical_frame" />
+    </joint>
+    <link name="camera_rgb_optical_frame"/>
+    <joint name="camera_joint" type="fixed">
 			<origin xyz="${joint_x} ${joint_y} ${joint_z}" rpy="${joint_roll} ${joint_pitch} ${joint_yaw}"/>
-			<parent link="${parent_link}"/>
-			<child link="${prefix}_link"/>
-		</joint>
-		<!-- Kinect Dummy Link -->
-		<link name="kinect_dummy">
-			<pose>0 0 0 0 0 0</pose>
-		</link>
-		<!-- Kinect Dummy Joint -->
-		<joint name="kinect_joint_dummy" type="fixed">
-			<origin xyz="0 0 0" rpy="-1.57 0.0 -1.57"/>
-			<parent link="${prefix}_link"/>
-			<child link="kinect_dummy"/>
-			<axis xyz="0 1 0"/>
-		</joint>
-		<!-- Kinect Gazebo Plugin -->
-		<gazebo reference="${prefix}_link">
-			<sensor type="depth" name="openni_camera_camera">
-				<always_on>1</always_on>
-				<visualize>false</visualize>
-				<camera>
-					<horizontal_fov>1.047</horizontal_fov>
-					<image>
-						<width>640</width>
-						<height>480</height>
-						<format>R8G8B8</format>
-					</image>
-					<depth_camera>
-					</depth_camera>
-					<clip>
-						<near>0.2</near>
-						<far>100</far>
-					</clip>
-				</camera>
-				<plugin name="${prefix}_controller" filename="libgazebo_ros_openni_kinect.so">
-					<baseline>${base_line}</baseline>
-					<alwaysOn>true</alwaysOn>
-					<updateRate>${update_rate}</updateRate>
-					<cameraName>${camera_name}</cameraName>
-					<imageTopicName>/${camera_name}/depth/image_raw</imageTopicName>
-					<depthImageCameraInfoTopicName>${camera_name}/depth/image_camera_info</depthImageCameraInfoTopicName>
-					<pointCloudCutoffMax>5.0</pointCloudCutoffMax>
-					<cameraInfoTopicName>/${camera_name}/depth/camera_info</cameraInfoTopicName>
-					<depthImageTopicName>/${camera_name}/depth/image_raw</depthImageTopicName>
-					<depthImageInfoTopicName>/${camera_name}/depth/camera_info</depthImageInfoTopicName>
-					<pointCloudTopicName>/${camera_name}/depth/points</pointCloudTopicName>
-					<frameName>kinect_dummy</frameName>
-					<pointCloudCutoff>0.5</pointCloudCutoff>
+      <parent link="${parent_link}"/>
+      <child link="camera_link"/>
+    </joint>
+    <link name="camera_link">
+      <visual>
+        <origin xyz="0.0 0.0 0.004" rpy="0 0 0"/>
+        <geometry>
+          <mesh filename="package://evarobot_description/meshes/xtion_pro_camera.dae"/>
+        </geometry>
+      </visual>
+      <collision>
+        <origin xyz="0.0 0.0 0.0" rpy="0 0 0" />
+        <geometry>
+        <box size="0.0730 0.2760 0.0720"/>
+      </geometry>
+      </collision>
+      <inertial>
+        <mass value="0.170" />
+        <origin xyz="0 0 0" />
+        <inertia ixx="0.001152600" ixy="0.0" ixz="0.0"
+                 iyy="0.000148934" iyz="0.0"
+                 izz="0.001154654" />
+      </inertial>
+    </link>
+    <joint name="camera_depth_joint" type="fixed">
+      <origin xyz="0 -0.045 0" rpy="0 0 0" />
+      <parent link="camera_link" />
+      <child link="camera_depth_frame" />
+    </joint>
+    <link name="camera_depth_frame"/>
+    <joint name="camera_depth_optical_joint" type="fixed">
+      <origin xyz="0 0 0" rpy="${-pi/2} 0 ${-pi/2}" />
+      <parent link="camera_depth_frame" />
+      <child link="camera_depth_optical_frame" />
+    </joint>
+    <link name="camera_depth_optical_frame"/>
+    <!-- Asus mount -->
+    <joint name="mount_asus_xtion_pro_joint" type="fixed">
+			<origin xyz="${0.17 -16.5/1000 + 0.015} -0.0050 ${0.21 - 18.7/1000 -35/1000}" rpy="${pi/2} 0 ${-pi/2}"/>
+      <parent link="base_link"/>
+      <child link="mount_asus_xtion_pro_link"/>
+    </joint>
+    <link name="mount_asus_xtion_pro_link">
+      <visual>
+        <origin xyz="0 0 0" rpy="0 0 0"/>
+        <geometry>
+          <mesh filename="package://evarobot_description/meshes/asus_base.stl"/>
+        </geometry>
+        <material name="Black"/>
+      </visual>
+      <collision>
+        <origin xyz="0.0 0.0 0.0" rpy="0 0 0" />
+        <geometry>
+        <box size="0.2760 0.0330 0.0120"/>
+      </geometry>
+      </collision>
+      <inertial>
+        <mass value="0.170" />
+        <origin xyz="0 0 0" />
+        <inertia ixx="0.001152600" ixy="0.0" ixz="0.0"
+                 iyy="0.000148934" iyz="0.0"
+                 izz="0.001154654" />
+      </inertial>
+    </link>
+		<gazebo reference="mount_asus_xtion_pro_link">
+			<material>Gazebo/Black</material>
+		</gazebo>
+		<gazebo reference="camera_link">
+      <sensor type="depth" name="camera">
+        <always_on>true</always_on>
+        <update_rate>20.0</update_rate>
+        <camera>
+          <horizontal_fov>${60.0*pi/180.0}</horizontal_fov>
+          <image>
+            <format>R8G8B8</format>
+            <width>640</width>
+            <height>480</height>
+          </image>
+          <clip>
+            <near>0.05</near>
+            <far>8.0</far>
+          </clip>
+        </camera>
+        <plugin name="kinect_camera_controller" filename="libgazebo_ros_openni_kinect.so">
+          <cameraName>camera</cameraName>
+          <alwaysOn>true</alwaysOn>
+          <updateRate>10</updateRate>
+          <imageTopicName>rgb/image_raw</imageTopicName>
+          <depthImageTopicName>depth/image_raw</depthImageTopicName>
+          <pointCloudTopicName>depth/points</pointCloudTopicName>
+          <cameraInfoTopicName>rgb/camera_info</cameraInfoTopicName>
+          <depthImageCameraInfoTopicName>depth/camera_info</depthImageCameraInfoTopicName>
+          <frameName>camera_depth_optical_frame</frameName>
+          <baseline>0.1</baseline>
+					<pointCloudCutoff>0.4</pointCloudCutoff>
 					<distortionK1>0.00000001</distortionK1>
 					<distortionK2>0.00000001</distortionK2>
@@ -89,7 +127,7 @@
 					<focalLength>0</focalLength>
 					<hackBaseline>0</hackBaseline>
-				</plugin>
-			</sensor>
-		</gazebo>
+        </plugin>
+      </sensor>
+    </gazebo>
 	</xacro:macro>
 </robot>

File: evarobot_description/urdf/evarobot_lidar.urdf.xacro (robot description, xacro)
@@ -14,11 +14,11 @@
 				</geometry>
 			</collision>
-<!--			<visual>
-				<origin xyz="0 0 0" rpy="0 0 0"/>
+			<visual>
+				<origin xyz="${-55/1000} ${-110/1000} ${-50/1000}" rpy="${-pi/2} ${pi} 0"/>
 				<geometry>
-					<mesh filename="package://evarobot_description/meshes/rplidar.stl" scale="0.01 0.01 0.01" />
+					<mesh filename="package://evarobot_description/meshes/rplidar.stl" scale="0.001 0.001 0.001" />
 				</geometry>
+				<material name="Black" />
 			</visual>
--->
 			<inertial>
 				<mass value="1e-5" />
@@ -34,4 +34,5 @@
 		</joint>
 		<gazebo reference="${prefix}_link">
+			<material>Gazebo/Black</material>
 			<sensor type="gpu_ray" name="head_hokuyo_sensor">
 				<pose>0 0 0 0 0 0</pose>
@@ -63,5 +64,4 @@
 				</ray>
     			<plugin name="${prefix}_controller" filename="libgazebo_ros_gpu_laser.so">
-					<robotNamespace>${robot_namespace}</robotNamespace>
 					<topicName>${topic_name}</topicName>
 					<frameName>${frame_name}</frameName>
@@ -69,9 +69,4 @@
 			</sensor>
 		</gazebo>
-		<gazebo>
-			<plugin name="${prefix}_control" filename="libgazebo_ros_control.so">
-				<robotNamespace>${robot_namespace}</robotNamespace>
-			</plugin>
-		</gazebo>
 	</xacro:macro>
 </robot>

File: evarobot_description/urdf/evarobot_sonar.urdf.xacro (robot description, xacro)
@@ -14,5 +14,5 @@
 				<mass value="0.001" />
 				<origin xyz="0 0 0" rpy="0 0 0" />
-				<inertia ixx="0.000000017" ixy="0" ixz="0" iyy="0.000000017" iyz="0" izz="0.000000017" />
+				<inertia ixx="1e-6" ixy="0" ixz="0" iyy="1e-6" iyz="0" izz="1e-6" />
 			</inertial>
 <!--			<visual>

File: evarobot_description/urdf/evarobot_wheel.urdf.xacro (robot description, xacro)
@@ -10,17 +10,28 @@
 			</collision>
 			<visual>
-				<origin rpy="1.57075 0 0" xyz="0 0 0"/>
+				<origin rpy="0 0 ${pi/2}" xyz="0 0 0"/>
 				<geometry>
-					<cylinder length="${cylinder_length}" radius="${cylinder_radius}"/>
-					<mesh filename="model://evarobot/meshes/wheel.stl" scale="0.001 0.001 0.001"/>
+					 <mesh filename="package://evarobot_description/meshes/rim.stl" scale="1 1 1"/>
 				</geometry>
-				<material name="black"/>
+				<material name="Grey"/>
 			</visual>
 			<inertial>
-				<origin xyz="0 0 0" rpy="0 0 0"/>
-				<mass value="0.75"/>
-				<inertia ixx="1e-2" ixy="0" ixz="0" iyy="1e-2" iyz="0" izz="1e-2" />
+				<origin rpy="1.57075 0 0" xyz="0 0 0"/>
+				<mass value="0.85"/>
+				<inertia
+					ixx="0.001" ixy="0" ixz="0"
+					iyy="0.001" iyz="0"
+					izz="0.001"/>
 			</inertial>
 		</link>
+		<gazebo reference="${prefix}_link">
+			<material>Gazebo/Grey</material>
+	    <mu1>1.0</mu1>
+	    <mu2>1.0</mu2>
+	    <kp>1000000.0</kp>
+	    <kd>100.0</kd>
+	    <minDepth>0.001</minDepth>
+	    <maxVel>1.0</maxVel>
+		</gazebo>
 		<joint name="${prefix}_joint" type="continuous">
 			<axis xyz="0 1 0"/>
@@ -28,6 +39,36 @@
 			<child link="${prefix}_link"/>
 			<origin rpy="${joint_roll} ${joint_pitch} ${joint_yaw}" xyz="${joint_x} ${joint_y} ${joint_z}"/>
-			<limit effort="100" velocity="100"/>
-			<joint_properties damping="0.0" friction="0.0"/>
+		</joint>
+		<link name="${prefix}tire_link">
+			<collision>
+				<origin rpy="1.57075 0 0" xyz="0 0 0"/>
+				<geometry>
+					<cylinder length="0.001" radius="0.001"/>
+				</geometry>
+			</collision>
+			<visual>
+				<origin rpy="0 0 ${pi/2}" xyz="0 0 0"/>
+				<geometry>
+					<mesh filename="package://evarobot_description/meshes/tire.stl" scale="1 1 1"/>
+				</geometry>
+				<material name="Black"/>
+			</visual>
+			<inertial>
+				<origin xyz="0 0 0" rpy="0 0 0"/>
+				<mass value="0.001"/>
+				<inertia
+					ixx="0.001" ixy="0" ixz="0"
+					iyy="0.001" iyz="0"
+					izz="0.001"/>
+			</inertial>
+		</link>
+		<gazebo reference="${prefix}tire_link">
+			<material>Gazebo/Black</material>
+		</gazebo>
+		<joint name="${prefix}tire_joint" type="continuous">
+			<axis xyz="0 1 0"/>
+			<parent link="${prefix}_link"/>
+			<child link="${prefix}tire_link"/>
+			<origin rpy="0 0 0" xyz="0.0 0.0 0.0"/>
 		</joint>
 	</xacro:macro>
